Commit message: fix/move it + mujoco pipeline

File: workspace/src/aesir_robot_description/urdf/rescue_robot.urdf.xacro (robot description, xacro)
@@ -75,5 +75,5 @@
     </inertial>
   </link>
-  <joint name="flipper_1_joint" type="revolute">
+  <joint name="flipper_joint_1" type="revolute">
     <parent link="base_link"/>
     <child link="flipper_1_link"/>
@@ -98,5 +98,5 @@
     </inertial>
   </link>
-  <joint name="flipper_2_joint" type="revolute">
+  <joint name="flipper_joint_2" type="revolute">
     <parent link="base_link"/>
     <child link="flipper_2_link"/>
@@ -121,5 +121,5 @@
     </inertial>
   </link>
-  <joint name="flipper_3_joint" type="revolute">
+  <joint name="flipper_joint_3" type="revolute">
     <parent link="base_link"/>
     <child link="flipper_3_link"/>
@@ -144,5 +144,5 @@
     </inertial>
   </link>
-  <joint name="flipper_4_joint" type="revolute">
+  <joint name="flipper_joint_4" type="revolute">
     <parent link="base_link"/>
     <child link="flipper_4_link"/>
@@ -150,4 +150,47 @@
     <axis xyz="0 1 0"/>
     <limit lower="-3.14" upper="3.14" effort="150.0" velocity="3.14"/>
+  </joint>
+  <!-- ================= DRIVE WHEELS (kinematic placeholders) ================= -->
+  <link name="drive_l_1_link"/>
+  <joint name="drive_l_1" type="continuous">
+    <parent link="base_link"/>
+    <child link="drive_l_1_link"/>
+    <origin xyz="-0.3 -0.25 -0.05" rpy="0 0 0"/>
+    <axis xyz="0 1 0"/>
+  </joint>
+  <link name="drive_l_2_link"/>
+  <joint name="drive_l_2" type="continuous">
+    <parent link="base_link"/>
+    <child link="drive_l_2_link"/>
+    <origin xyz="0.0 -0.25 -0.05" rpy="0 0 0"/>
+    <axis xyz="0 1 0"/>
+  </joint>
+  <link name="drive_l_3_link"/>
+  <joint name="drive_l_3" type="continuous">
+    <parent link="base_link"/>
+    <child link="drive_l_3_link"/>
+    <origin xyz="0.3 -0.25 -0.05" rpy="0 0 0"/>
+    <axis xyz="0 1 0"/>
+  </joint>
+  <link name="drive_r_1_link"/>
+  <joint name="drive_r_1" type="continuous">
+    <parent link="base_link"/>
+    <child link="drive_r_1_link"/>
+    <origin xyz="-0.3 0.25 -0.05" rpy="0 0 0"/>
+    <axis xyz="0 1 0"/>
+  </joint>
+  <link name="drive_r_2_link"/>
+  <joint name="drive_r_2" type="continuous">
+    <parent link="base_link"/>
+    <child link="drive_r_2_link"/>
+    <origin xyz="0.0 0.25 -0.05" rpy="0 0 0"/>
+    <axis xyz="0 1 0"/>
+  </joint>
+  <link name="drive_r_3_link"/>
+  <joint name="drive_r_3" type="continuous">
+    <parent link="base_link"/>
+    <child link="drive_r_3_link"/>
+    <origin xyz="0.3 0.25 -0.05" rpy="0 0 0"/>
+    <axis xyz="0 1 0"/>
   </joint>
   <!-- ================= BASE ARM ================= -->

File: workspace/src/robot_moveit_config/config/rescue_robot.ros2_control.xacro (robot description, xacro)
@@ -1,27 +1,10 @@
 <?xml version="1.0"?>
 <robot xmlns:xacro="http://www.ros.org/wiki/xacro">
-    <xacro:macro name="rescue_robot_ros2_control" params="name initial_positions_file">
-        <xacro:property name="initial_positions" value="${load_yaml(initial_positions_file)['initial_positions']}"/>
+    <xacro:macro name="rescue_robot_ros2_control" params="name initial_positions_file mujoco_model:=''">
+        <xacro:property name="initial_positions" value="${xacro.load_yaml(initial_positions_file)['initial_positions']}"/>
         <ros2_control name="${name}" type="system">
             <hardware>
-                <!--
-                    HARDWARE PLUGIN
-                    ===============
-                    Active plugin: mujoco_ros2_control/MujocoSystem
-                        Reads command interfaces from this <ros2_control> block
-                        and writes them as ctrl values on the MuJoCo model
-                        loaded by the mujoco_ros2_control node. State
-                        interfaces are populated from MuJoCo's qpos / qvel /
-                        sensor data each control cycle.
-                    Disconnected: aesir_plugin/TopicBridgeHardware
-                        The custom topic-bridge plugin is intentionally
-                        commented out below. Re-enable ONLY if you go back
-                        to the topic-bridge integration path; in that case
-                        you must also re-enable its build targets in
-                        robot_moveit_config/CMakeLists.txt and the export
-                        in robot_moveit_config/package.xml.
-                -->
-                <plugin>mujoco_ros2_control/MujocoSystem</plugin>
-                <!-- <plugin>aesir_plugin/TopicBridgeHardware</plugin> -->
+                <plugin>mujoco_ros2_control/MujocoSystemInterface</plugin>
+                <param name="mujoco_model">${mujoco_model}</param>
             </hardware>
             <joint name="joint_1">
@@ -85,27 +68,58 @@
                 <state_interface name="effort"/>
             </joint>
-            <joint name="flipper_1_joint">
+            <joint name="flipper_joint_1">
                 <command_interface name="position"/>
                 <state_interface name="position">
-                    <param name="initial_value">${initial_positions['flipper_1_joint']}</param>
+                    <param name="initial_value">${initial_positions['flipper_joint_1']}</param>
                 </state_interface>
             </joint>
-            <joint name="flipper_2_joint">
+            <joint name="flipper_joint_2">
                 <command_interface name="position"/>
                 <state_interface name="position">
-                    <param name="initial_value">${initial_positions['flipper_2_joint']}</param>
+                    <param name="initial_value">${initial_positions['flipper_joint_2']}</param>
                 </state_interface>
             </joint>
-            <joint name="flipper_3_joint">
+            <joint name="flipper_joint_3">
                 <command_interface name="position"/>
                 <state_interface name="position">
-                    <param name="initial_value">${initial_positions['flipper_3_joint']}</param>
+                    <param name="initial_value">${initial_positions['flipper_joint_3']}</param>
                 </state_interface>
             </joint>
-            <joint name="flipper_4_joint">
+            <joint name="flipper_joint_4">
                 <command_interface name="position"/>
                 <state_interface name="position">
-                    <param name="initial_value">${initial_positions['flipper_4_joint']}</param>
+                    <param name="initial_value">${initial_positions['flipper_joint_4']}</param>
                 </state_interface>
+            </joint>
+            <!-- Drive wheel joints (left 1-3, right 1-3) — velocity only for diff_drive_controller -->
+            <joint name="drive_l_1">
+                <command_interface name="velocity"/>
+                <state_interface name="position"/>
+                <state_interface name="velocity"/>
+            </joint>
+            <joint name="drive_l_2">
+                <command_interface name="velocity"/>
+                <state_interface name="position"/>
+                <state_interface name="velocity"/>
+            </joint>
+            <joint name="drive_l_3">
+                <command_interface name="velocity"/>
+                <state_interface name="position"/>
+                <state_interface name="velocity"/>
+            </joint>
+            <joint name="drive_r_1">
+                <command_interface name="velocity"/>
+                <state_interface name="position"/>
+                <state_interface name="velocity"/>
+            </joint>
+            <joint name="drive_r_2">
+                <command_interface name="velocity"/>
+                <state_interface name="position"/>
+                <state_interface name="velocity"/>
+            </joint>
+            <joint name="drive_r_3">
+                <command_interface name="velocity"/>
+                <state_interface name="position"/>
+                <state_interface name="velocity"/>
             </joint>
         </ros2_control>

File: workspace/src/robot_moveit_config/config/rescue_robot.urdf.xacro (robot description, xacro)
@@ -2,8 +2,13 @@
 <robot xmlns:xacro="http://www.ros.org/wiki/xacro" name="rescue_robot">
     <xacro:arg name="initial_positions_file" default="initial_positions.yaml" />
+    <!-- Path to MuJoCo MJCF scene. Set at launch time via xacro mappings. -->
+    <xacro:arg name="mujoco_model" default="" />
     <!-- Import rescue_robot urdf file -->
     <xacro:include filename="$(find aesir_robot_description)/urdf/rescue_robot.urdf.xacro" />
     <!-- Import control_xacro -->
     <xacro:include filename="rescue_robot.ros2_control.xacro" />
-    <xacro:rescue_robot_ros2_control name="FakeSystem" initial_positions_file="$(arg initial_positions_file)"/>
+    <xacro:rescue_robot_ros2_control
+        name="FakeSystem"
+        initial_positions_file="$(arg initial_positions_file)"
+        mujoco_model="$(arg mujoco_model)"/>
 </robot>
