Commit message: Arm kinematics working - Updated to new model the robot_moveit_config package - Controller manager for gripper - Fix bugs of urdf model - Little updated of initial positions

File: ros2_ws/src/aesir_robot_description/urdf/rescue_robot_v2.urdf.xacro (robot description, xacro)
@@ -11,18 +11,11 @@
   <xacro:property name="L_TOOL" value="0.28450"/>
   <xacro:property name="L_TOOL_END" value="${L_TOOL-L_WRIST_END}"/>
-  <!-- ============== INITIAL POSITIONS ============== -->
-  <xacro:property name="INIT_J1" value="0.0"/>
-  <xacro:property name="INIT_J2" value="-2.86234"/>
-  <xacro:property name="INIT_J3" value="2.86234"/>
-  <xacro:property name="INIT_J4" value="-1.5708"/>
-  <xacro:property name="INIT_J5" value="-1.5708"/>
-  <xacro:property name="INIT_J6" value="0.0"/>
-  <xacro:property name="INIT_FLIP" value="0.0"/>
   <!-- ================= MATERIALES ================= -->
   <material name="gray"><color rgba="0.7 0.7 0.7 1.0"/></material>
   <material name="orange"><color rgba="1.0 0.4 0.0 1.0"/></material>
   <material name="black"><color rgba="0.2 0.2 0.2 1.0"/></material>
+  <material name="silver"><color rgba="0.75 0.75 0.75 1.0"/></material>
   <!-- ================= BASE ROBOT ================= -->
-  <link name="world">
+  <link name="base_footprint">
     <visual>
       <geometry>
@@ -31,39 +24,68 @@
     </visual>
   </link>
-  <joint name="world_to_base" type="fixed">
-    <parent link="world"/>
-    <child link="base_link"/>
-    <origin xyz="0 0 0" rpy="0 0 0"/>
-  </joint>
-  <link name="base_footprint">
-    <visual>
-      <geometry>
-        <box size="0.001 0.001 0.001"/>
-      </geometry>
-    </visual>
-  </link>
   <joint name="base_to_base_footprint" type="fixed">
     <parent link="base_link"/>
     <child link="base_footprint"/>
-    <origin xyz="0 0 -0.09" rpy="0 0 0"/>
+    <origin xyz="0 0 -0.03" rpy="0 0 0"/>
   </joint>
   <link name="base_link">
-    <visual>
-      <origin rpy="0 0 0" xyz="0 0.757 0"/>
+    <inertial>
+      <origin xyz="0 0 0" rpy="0 0 0"/>
+      <mass value="25"/>
+      <inertia ixx="1.238151" iyy="1.620218" izz="2.702376" ixy="0.0" iyz="-0.0" ixz="0.0"/>
+    </inertial>
+    <visual>
+      <origin xyz="0 0.55 0" rpy="0 0 0"/>
       <geometry>
         <mesh filename="package://aesir_robot_description/meshes/base_link.stl" scale="0.001 0.001 0.001"/>
       </geometry>
-    </visual>
-    <collision>
-      <origin rpy="0 0 0" xyz="0 0.757 0."/>
+      <material name="silver"/>
+    </visual>
+    <collision>
+      <origin xyz="0 0.55 0" rpy="0 0 0"/>
       <geometry>
         <mesh filename="package://aesir_robot_description/meshes/base_link.stl" scale="0.001 0.001 0.001"/>
       </geometry>
     </collision>
-    <inertial>
-      <origin rpy="0 0 0" xyz="0 0.757 0"/>
-      <mass value="5.0"/>
-      <inertia ixx="0.2" ixy="0" ixz="0" iyy="0.2" iyz="0" izz="0.2"/>
-    </inertial>
+  </link>
+  <link name="tracked_1_link">
+    <inertial>
+      <origin xyz="0 0 0" rpy="0 0 0"/>
+      <mass value="3.5"/>
+      <inertia ixx="0.064824" iyy="0.377269" izz="0.351452" ixy="0.0" iyz="-0.0" ixz="-0.0"/>
+    </inertial>
+    <visual>
+      <origin xyz="0.24 0.806 -0.06" rpy="0 0 0"/>
+      <geometry>
+        <mesh filename="package://aesir_robot_description/meshes/tracked_1.stl" scale="0.001 0.001 0.001"/>
+      </geometry>
+      <material name="silver"/>
+    </visual>
+    <collision>
+      <origin xyz="0.24 0.806 -0.06" rpy="0 0 0"/>
+      <geometry>
+        <mesh filename="package://aesir_robot_description/meshes/tracked_1.stl" scale="0.001 0.001 0.001"/>
+      </geometry>
+    </collision>
+  </link>
+  <link name="tracked_2_link">
+    <inertial>
+      <origin xyz="0 0 0" rpy="0 0 0"/>
+      <mass value="3.5"/>
+      <inertia ixx="0.064824" iyy="0.377269" izz="0.351452" ixy="0.0" iyz="0.0" ixz="-0.0"/>
+    </inertial>
+    <visual>
+      <origin xyz="0.24 0.306 -0.06" rpy="0 0 0"/>
+      <geometry>
+        <mesh filename="package://aesir_robot_description/meshes/tracked_2.stl" scale="0.001 0.001 0.001"/>
+      </geometry>
+      <material name="silver"/>
+    </visual>
+    <collision>
+      <origin xyz="0.24 0.306 -0.06" rpy="0 0 0"/>
+      <geometry>
+        <mesh filename="package://aesir_robot_description/meshes/tracked_2.stl" scale="0.001 0.001 0.001"/>
+      </geometry>
+    </collision>
   </link>
   <!-- ================= SENSORS ================= -->
@@ -90,5 +112,5 @@
     <parent link="base_link"/>
     <child link="lidar_link"/>
-    <origin xyz="0.357 0 0.09" rpy="0 0.785398 0"/>
+    <origin xyz="0.320 0 0.105" rpy="0 0.785398 0"/>
   </joint>
   <link name="oakd_link">
@@ -112,9 +134,9 @@
     <parent link="base_link"/>
     <child link="oakd_link"/>
-    <origin xyz="0.257 0 0.15" rpy="0 0 0"/>
+    <origin xyz="0.257 0 0.17" rpy="0 0 0"/>
   </joint>
   <link name="arm_camera_link">
     <visual>
-      <origin rpy="0 0 -1.5708" xyz="0 0.05 -0.2"/>
+      <origin rpy="0 0 -1.5708" xyz="0.02 0.04 -0.2"/>
       <geometry>
         <mesh filename="package://aesir_robot_description/meshes/logitech_c920.stl" scale="0.001 0.001 0.001"/>
@@ -123,5 +145,5 @@
     </visual>
     <collision>
-      <origin rpy="0 0 -1.5708" xyz="0 0.05 -0.2"/>
+      <origin rpy="0 0 -1.5708" xyz="0.02 0.04 -0.2"/>
       <geometry>
         <mesh filename="package://aesir_robot_description/meshes/logitech_c920.stl" scale="0.001 0.001 0.001"/>
@@ -136,5 +158,5 @@
     <parent link="link_6"/>
     <child link="arm_camera_link"/>
-    <origin xyz="0 -0.03 0.06" rpy="-0.174533 0 0"/>
+    <origin xyz="0 0 0.06" rpy="-0.174533 0 0"/>
   </joint>
   <link name="back_camera_link">
@@ -160,97 +182,124 @@
     <parent link="base_link"/>
     <child link="back_camera_link"/>
-    <origin xyz="-0.35 0 0.1" rpy="0 0 3.14159"/>
+    <origin xyz="-0.30 0 0.17" rpy="0 0 3.14159"/>
   </joint>
   <!-- ================= FLIPPER 1 ================= -->
   <link name="flipper_1_link">
-    <visual>
-      <origin rpy="0 0 0" xyz="0.3 1.06 0"/>
-      <geometry><mesh filename="package://aesir_robot_description/meshes/flipper_1_1.stl" scale="0.001 0.001 0.001"/></geometry>
-    </visual>
-    <collision>
-      <origin rpy="0 0 0" xyz="0.3 1.06 0"/>
-      <geometry><mesh filename="package://aesir_robot_description/meshes/flipper_1_1.stl" scale="0.001 0.001 0.001"/></geometry>
-    </collision>
-    <inertial>
-      <origin rpy="0 0 0" xyz="0.3 1.06 0"/>
-      <mass value="0.8"/>
-      <inertia ixx="0.01" ixy="0" ixz="0" iyy="0.02" iyz="0" izz="0.02"/>
-    </inertial>
-  </link>
-  <joint name="flipper_1_joint" type="revolute">
-    <parent link="base_link"/>
-    <child link="flipper_1_link"/>
-    <origin rpy="0 0 0" xyz="-0.3 0.3 0"/>
-    <axis xyz="0 1 0"/>
-    <limit lower="-3.14" upper="3.14" effort="150.0" velocity="3.14"/>
-  </joint>
+    <inertial>
+      <origin xyz="5.551115123125783e-17 0.003554085914685201 0.15154044804505273" rpy="0 0 0"/>
+      <mass value="3.742066453745571"/>
+      <inertia ixx="0.065573" iyy="0.072966" izz="0.008972" ixy="0.0" iyz="-0.00082" ixz="-0.0"/>
+    </inertial>
+    <visual>
+      <origin xyz="0.24 0.836 -0.06" rpy="0 0 0"/>
+      <geometry>
+        <mesh filename="package://aesir_robot_description/meshes/flipper_1_1.stl" scale="0.001 0.001 0.001"/>
+      </geometry>
+      <material name="silver"/>
+    </visual>
+    <collision>
+      <origin xyz="0.24 0.836 -0.06" rpy="0 0 3.14159"/>
+      <geometry>
+        <mesh filename="package://aesir_robot_description/meshes/flipper_1_1.stl" scale="0.001 0.001 0.001"/>
+      </geometry>
+    </collision>
+  </link>
   <!-- ================= FLIPPER 2 ================= -->
   <link name="flipper_2_link">
-    <visual>
-      <origin rpy="0 0 0" xyz="0.3 0.45 0"/>
-      <geometry><mesh filename="package://aesir_robot_description/meshes/flipper_2_1.stl" scale="0.001 0.001 0.001"/></geometry>
-    </visual>
-    <collision>
-      <origin rpy="0 0 0" xyz="0.3 0.45 0"/>
-      <geometry><mesh filename="package://aesir_robot_description/meshes/flipper_2_1.stl" scale="0.001 0.001 0.001"/></geometry>
-    </collision>
-    <inertial>
-      <origin rpy="0 0 0" xyz="0.3 0.45 0"/>
-      <mass value="0.8"/>
-      <inertia ixx="0.01" ixy="0" ixz="0" iyy="0.02" iyz="0" izz="0.02"/>
-    </inertial>
-  </link>
-  <joint name="flipper_2_joint" type="revolute">
-    <parent link="base_link"/>
-    <child link="flipper_2_link"/>
-    <origin rpy="0 0 0" xyz="-0.3 -0.3 0"/>
-    <axis xyz="0 1 0"/>
-    <limit lower="-3.14" upper="3.14" effort="150.0" velocity="3.14"/>
-  </joint>
+    <inertial>
+      <origin xyz="-2.7755575615628914e-17 -0.0035540859146853676 0.15154044804505265" rpy="0 0 0"/>
+      <mass value="3.7420664537455717"/>
+      <inertia ixx="0.065573" iyy="0.072966" izz="0.008972" ixy="0.0" iyz="0.00082" ixz="0.0"/>
+    </inertial>
+    <visual>
+      <origin xyz="-0.24 0.276 -0.06" rpy="0 0 0"/>
+      <geometry>
+        <mesh filename="package://aesir_robot_description/meshes/flipper_4_1.stl" scale="0.001 0.001 0.001"/>
+      </geometry>
+      <material name="silver"/>
+    </visual>
+    <collision>
+      <origin xyz="-0.24 0.276 -0.06" rpy="0 0 0"/>
+      <geometry>
+        <mesh filename="package://aesir_robot_description/meshes/flipper_4_1.stl" scale="0.001 0.001 0.001"/>
+      </geometry>
+    </collision>
+  </link>
   <!-- ================= FLIPPER 3 ================= -->
   <link name="flipper_3_link">
-    <visual>
-      <origin rpy="0 0 0" xyz="-0.3 1.06 0"/>
-      <geometry><mesh filename="package://aesir_robot_description/meshes/flipper_3_1.stl" scale="0.001 0.001 0.001"/></geometry>
-    </visual>
-    <collision>
-      <origin rpy="0 0 0" xyz="-0.3 1.06 0"/>
-      <geometry><mesh filename="package://aesir_robot_description/meshes/flipper_3_1.stl" scale="0.001 0.001 0.001"/></geometry>
-    </collision>
-    <inertial>
-      <origin rpy="0 0 0" xyz="-0.3 1.06 0"/>
-      <mass value="0.8"/>
-      <inertia ixx="0.01" ixy="0" ixz="0" iyy="0.02" iyz="0" izz="0.02"/>
-    </inertial>
-  </link>
-  <joint name="flipper_3_joint" type="revolute">
-    <parent link="base_link"/>
-    <child link="flipper_3_link"/>
-    <origin rpy="0 0 0" xyz="0.3 0.3 0"/>
-    <axis xyz="0 1 0"/>
-    <limit lower="-3.14" upper="3.14" effort="150.0" velocity="3.14"/>
-  </joint>
+    <inertial>
+      <origin xyz="5.551115123125783e-17 -0.0035540859146853676 0.15154044804505276" rpy="0 0 0"/>
+      <mass value="3.7420664537455717"/>
+      <inertia ixx="0.065573" iyy="0.072966" izz="0.008972" ixy="-0.0" iyz="0.00082" ixz="0.0"/>
+    </inertial>
+    <visual>
+      <origin xyz="0.24 0.276 -0.06" rpy="0 0 0"/>
+      <geometry>
+        <mesh filename="package://aesir_robot_description/meshes/flipper_3_1.stl" scale="0.001 0.001 0.001"/>
+      </geometry>
+      <material name="silver"/>
+    </visual>
+    <collision>
+      <origin xyz="0.24 0.276 -0.06" rpy="0 0 0"/>
+      <geometry>
+        <mesh filename="package://aesir_robot_description/meshes/flipper_3_1.stl" scale="0.001 0.001 0.001"/>
+      </geometry>
+    </collision>
+  </link>
   <!-- ================= FLIPPER 4 ================= -->
   <link name="flipper_4_link">
-    <visual>
-      <origin rpy="0 0 0" xyz="-0.3 0.45 0"/>
-      <geometry><mesh filename="package://aesir_robot_description/meshes/flipper_4_1.stl" scale="0.001 0.001 0.001"/></geometry>
-    </visual>
-    <collision>
-      <origin rpy="0 0 0" xyz="-0.3 0.45 0"/>
-      <geometry><mesh filename="package://aesir_robot_description/meshes/flipper_4_1.stl" scale="0.001 0.001 0.001"/></geometry>
-    </collision>
-    <inertial>
-      <origin rpy="0 0 0" xyz="-0.3 0.45 0"/>
-      <mass value="0.8"/>
-      <inertia ixx="0.01" ixy="0" ixz="0" iyy="0.02" iyz="0" izz="0.02"/>
-    </inertial>
-  </link>
-  <joint name="flipper_4_joint" type="revolute">
+    <inertial>
+      <origin xyz="-2.7755575615628914e-17 -0.0035540859146853676 0.15154044804505265" rpy="0 0 0"/>
+      <mass value="3.7420664537455717"/>
+      <inertia ixx="0.065573" iyy="0.072966" izz="0.008972" ixy="0.0" iyz="0.00082" ixz="0.0"/>
+    </inertial>
+    <visual>
+      <origin xyz="-0.24 0.276 -0.06" rpy="0 0 0"/>
+      <geometry>
+        <mesh filename="package://aesir_robot_description/meshes/flipper_4_1.stl" scale="0.001 0.001 0.001"/>
+      </geometry>
+      <material name="silver"/>
+    </visual>
+    <collision>
+      <origin xyz="-0.24 0.276 -0.06" rpy="0 0 0"/>
+      <geometry>
+        <mesh filename="package://aesir_robot_description/meshes/flipper_4_1.stl" scale="0.001 0.001 0.001"/>
+      </geometry>
+    </collision>
+  </link>
+  <!-- ================= JOINTS BASE AND FLIPPERS ================= -->
+  <joint name="Rigid 1" type="fixed">
+    <origin xyz="-0.24 -0.256 0.06" rpy="0 0 0"/>
+    <parent link="base_link"/>
+    <child link="tracked_1_link"/>
+  </joint>
+  <joint name="Rigid 2" type="fixed">
+    <origin xyz="-0.24 0.256 0.06" rpy="0 0 0"/>
+    <parent link="base_link"/>
+    <child link="tracked_2_link"/>
+  </joint>
+  <joint name="flipper_1_joint" type="continuous">
+    <origin xyz="-0.24 -0.256 0.06" rpy="0 0 0"/>
+    <parent link="base_link"/>
+    <child link="flipper_1_link"/>
+    <axis xyz="0.0 -1.0 0.0"/>
+  </joint>
+  <joint name="flipper_2_joint" type="continuous">
+    <origin xyz="0.24 -0.256 0.06" rpy="0 0 0"/>
+    <parent link="base_link"/>
+    <child link="flipper_2_link"/>
+    <axis xyz="0.0 -1.0 0.0"/>
+  </joint>
+  <joint name="flipper_3_joint" type="continuous">
+    <origin xyz="0.24 0.256 0.06" rpy="0 0 0"/>
     <parent link="base_link"/>
     <child link="flipper_4_link"/>
-    <origin rpy="0 0 0" xyz="0.3 -0.3 0"/>
-    <axis xyz="0 1 0"/>
-    <limit lower="-3.14" upper="3.14" effort="150.0" velocity="3.14"/>
+    <axis xyz="0.0 1.0 0.0"/>
+  </joint>
+  <joint name="flipper_4_joint" type="continuous">
+    <origin xyz="-0.24 0.256 0.06" rpy="0 0 0"/>
+    <parent link="base_link"/>
+    <child link="flipper_3_link"/>
+    <axis xyz="0.0 1.0 0.0"/>
   </joint>
   <!-- ================= BASE ARM ================= -->
@@ -258,5 +307,5 @@
     <parent link="base_link"/>
     <child link="arm_base_link"/>
-    <origin xyz="0.12 0 0.04" rpy="0 0 0"/>
+    <origin xyz="0.12 0 0.06" rpy="0 0 0"/>
   </joint>
   <link name="arm_base_link">
@@ -439,4 +488,9 @@
     </inertial>
   </link>
+  <link name="tool_link"/>
+  <joint name="tool_joint" type="fixed">
+    <parent link="link_6"/>
+    <child link="tool_link"/> <origin xyz="0 0.12 0" rpy="0 0 1.5708"/>
+  </joint>
     <!-- ================= GRIPPER ================= -->
   <link name="gripper_base_link">

File: ros2_ws/src/robot_moveit_config/config/rescue_robot.ros2_control.xacro (robot description, xacro)
@@ -1,10 +1,10 @@
 <?xml version="1.0"?>
 <robot xmlns:xacro="http://www.ros.org/wiki/xacro">
-    <xacro:macro name="rescue_robot_ros2_control" params="name initial_positions_file mujoco_model:=''">
-        <xacro:property name="initial_positions" value="${xacro.load_yaml(initial_positions_file)['initial_positions']}"/>
+    <xacro:macro name="rescue_robot_ros2_control" params="name initial_positions_file">
+        <xacro:property name="initial_positions" value="${load_yaml(initial_positions_file)['initial_positions']}"/>
         <ros2_control name="${name}" type="system">
             <hardware>
-                <plugin>mujoco_ros2_control/MujocoSystemInterface</plugin>
-                <param name="mujoco_model">${mujoco_model}</param>
+                <!-- By default, set up controllers for simulation. This won't work on real hardware -->
+                <plugin>aesir_plugin/TopicBridgeHardware</plugin>
             </hardware>
             <joint name="joint_1">
@@ -68,58 +68,39 @@
                 <state_interface name="effort"/>
             </joint>
-            <joint name="flipper_joint_1">
+            <joint name="flipper_1_joint">
                 <command_interface name="position"/>
                 <state_interface name="position">
-                    <param name="initial_value">${initial_positions['flipper_joint_1']}</param>
+                    <param name="initial_value">${initial_positions['flipper_1_joint']}</param>
                 </state_interface>
             </joint>
-            <joint name="flipper_joint_2">
+            <joint name="flipper_2_joint">
                 <command_interface name="position"/>
                 <state_interface name="position">
-                    <param name="initial_value">${initial_positions['flipper_joint_2']}</param>
+                    <param name="initial_value">${initial_positions['flipper_2_joint']}</param>
                 </state_interface>
             </joint>
-            <joint name="flipper_joint_3">
+            <joint name="flipper_3_joint">
                 <command_interface name="position"/>
                 <state_interface name="position">
-                    <param name="initial_value">${initial_positions['flipper_joint_3']}</param>
+                    <param name="initial_value">${initial_positions['flipper_3_joint']}</param>
                 </state_interface>
             </joint>
-            <joint name="flipper_joint_4">
+            <joint name="flipper_4_joint">
                 <command_interface name="position"/>
                 <state_interface name="position">
-                    <param name="initial_value">${initial_positions['flipper_joint_4']}</param>
+                    <param name="initial_value">${initial_positions['flipper_4_joint']}</param>
                 </state_interface>
             </joint>
-            <!-- Drive wheel joints (left 1-3, right 1-3) — velocity only for diff_drive_controller -->
-            <joint name="drive_l_1">
-                <command_interface name="velocity"/>
-                <state_interface name="position"/>
-                <state_interface name="velocity"/>
+            <joint name="left_finger_joint">
+                <command_interface name="position"/>
+                <state_interface name="position">
+                    <param name="initial_value">${initial_positions['left_finger_joint']}</param>
+                </state_interface>
             </joint>
-            <joint name="drive_l_2">
-                <command_interface name="velocity"/>
-                <state_interface name="position"/>
-                <state_interface name="velocity"/>
-            </joint>
-            <joint name="drive_l_3">
-                <command_interface name="velocity"/>
-                <state_interface name="position"/>
-                <state_interface name="velocity"/>
-            </joint>
-            <joint name="drive_r_1">
-                <command_interface name="velocity"/>
-                <state_interface name="position"/>
-                <state_interface name="velocity"/>
-            </joint>
-            <joint name="drive_r_2">
-                <command_interface name="velocity"/>
-                <state_interface name="position"/>
-                <state_interface name="velocity"/>
-            </joint>
-            <joint name="drive_r_3">
-                <command_interface name="velocity"/>
-                <state_interface name="position"/>
-                <state_interface name="velocity"/>
+            <joint name="right_finger_joint">
+                <command_interface name="position"/>
+                <state_interface name="position">
+                    <param name="initial_value">${initial_positions['right_finger_joint']}</param>
+                </state_interface>
             </joint>
         </ros2_control>

File: ros2_ws/src/robot_moveit_config/config/rescue_robot.urdf.xacro (robot description, xacro)
@@ -2,13 +2,8 @@
 <robot xmlns:xacro="http://www.ros.org/wiki/xacro" name="rescue_robot">
     <xacro:arg name="initial_positions_file" default="initial_positions.yaml" />
-    <!-- Path to MuJoCo MJCF scene. Set at launch time via xacro mappings. -->
-    <xacro:arg name="mujoco_model" default="" />
     <!-- Import rescue_robot urdf file -->
-    <xacro:include filename="$(find aesir_robot_description)/urdf/rescue_robot.urdf.xacro" />
+    <xacro:include filename="$(find aesir_robot_description)/urdf/rescue_robot_v2.urdf.xacro" />
     <!-- Import control_xacro -->
     <xacro:include filename="rescue_robot.ros2_control.xacro" />
-    <xacro:rescue_robot_ros2_control
-        name="FakeSystem"
-        initial_positions_file="$(arg initial_positions_file)"
-        mujoco_model="$(arg mujoco_model)"/>
+    <xacro:rescue_robot_ros2_control name="FakeSystem" initial_positions_file="$(arg initial_positions_file)"/>
 </robot>
