Commit message: Update model robot - Fix position and orientaion of cameras - Add oak d mesh - Improve the number of wheels that simulate the tracked

File: ros2_ws/src/aesir_robot_description/urdf/rescue_robot_v2.urdf.xacro (robot description, xacro)
@@ -112,20 +112,22 @@
     <parent link="base_link"/>
     <child link="lidar_link"/>
-    <origin xyz="0.320 0 0.105" rpy="0 0.785398 0"/>
+    <origin xyz="0.305 0 0.112" rpy="0 0.785398 0"/>
   </joint>
   <link name="oakd_link">
     <visual>
-      <geometry>
-        <box size="0.02 0.1 0.03"/>
-      </geometry>
-      <material name="gray"/>
-    </visual>
-    <collision>
-      <geometry>
-        <box size="0.02 0.1 0.03"/>
-      </geometry>
-    </collision>
-    <inertial>
-      <mass value="0.1"/>
+      <origin xyz="0 0 0" rpy="1.5708 0 1.5708"/>
+      <geometry>
+        <mesh filename="package://aesir_robot_description/meshes/OAK-D-parts-14sep2020.stl" scale="0.001 0.001 0.001"/>
+      </geometry>
+      <material name="black"/>
+    </visual>
+    <collision>
+      <origin xyz="0 0 0" rpy="0 0 0"/>
+      <geometry>
+        <mesh filename="package://aesir_robot_description/meshes/OAK-D-parts-14sep2020.stl" scale="0.001 0.001 0.001"/>
+      </geometry>
+    </collision>
+    <inertial>
+      <mass value="0.182"/>
       <inertia ixx="0.0001" ixy="0" ixz="0" iyy="0.0001" iyz="0" izz="0.0001"/>
     </inertial>
@@ -134,9 +136,9 @@
     <parent link="base_link"/>
     <child link="oakd_link"/>
-    <origin xyz="0.257 0 0.17" rpy="0 0 0"/>
+    <origin xyz="0.257 0 0.19" rpy="0 0 0"/>
   </joint>
   <link name="arm_camera_link">
     <visual>
-      <origin rpy="0 0 -1.5708" xyz="0.02 0.04 -0.2"/>
+      <origin rpy="0 0 -1.5708" xyz="0.027 0.04 -0.2"/>
       <geometry>
         <mesh filename="package://aesir_robot_description/meshes/logitech_c920.stl" scale="0.001 0.001 0.001"/>
@@ -145,5 +147,5 @@
     </visual>
     <collision>
-      <origin rpy="0 0 -1.5708" xyz="0.02 0.04 -0.2"/>
+      <origin rpy="0 0 -1.5708" xyz="0.027 0.04 -0.2"/>
       <geometry>
         <mesh filename="package://aesir_robot_description/meshes/logitech_c920.stl" scale="0.001 0.001 0.001"/>
